Commit message: minor fixes

File: models/prometheus/urdf/gz.xacro (robot description, xacro)
@@ -55,4 +55,10 @@
                             <max_angle>${radians(two_d_lidar_max_angle)}</max_angle>
                         </horizontal>
+                        <!-- <vertical>
+                            <samples>360</samples>
+                            <resolution>1</resolution>
+                            <min_angle>${-7.22/180*3.1415926}</min_angle>
+                            <max_angle>${55.22/180*3.1415926}</max_angle>
+                        </vertical> -->
                     </scan>
                     <range>
@@ -99,5 +105,5 @@
         <sensor name="imu_sensor" type="imu">
             <always_on>1</always_on>
-            <update_rate>1</update_rate>
+            <update_rate>100</update_rate>
             <gz_frame_id>imu_frame</gz_frame_id>
             <visualize>true</visualize>

File: models/prometheus/urdf/prometheus.xacro (robot description, xacro)
@@ -15,5 +15,5 @@
     <xacro:property name="trolley_wheel_radius" value="0.03"/>
     <!-- a small constant -->
-    <xacro:property name="eps" value="0.002"/>
+    <xacro:property name="eps" value="0.0002"/>
     <xacro:property name="traction_wheel_radius" value="0.05"/>
     <xacro:property name="traction_wheel_width" value="0.03"/>
@@ -41,4 +41,5 @@
     <xacro:include filename="$(find prometheus)/models/prometheus/urdf/materials.xacro"/>
     <xacro:include filename="$(find prometheus)/models/prometheus/urdf/macros.xacro"/>
+    <!-- <xacro:include filename="$(find prometheus)/models/prometheus/urdf/mid360.xacro" /> -->
     <xacro:if value="$(arg arm_enabled)">
         <xacro:include filename="$(find prometheus)/models/so_100_arm_5dof/urdf/so_100_arm_5dof.urdf"/>

Commit message: fix nav2 cmd_vel pipeline and DiffDrive parameter mismatches
Remove cmd_vel from base remappings to fix ROS2 first-match-wins
issue where all nav2 nodes published directly to prometheus/cmd_vel,
bypassing velocity smoother and collision monitor. Set collision
monitor to publish directly to prometheus/cmd_vel. Make cmd_vel
bridge unidirectional (ROS2→GZ only). Fix wheel track width and
increase odom publish frequency. Add RotationShimController and
tune RPP/planner params.

File: models/prometheus/urdf/gz.xacro (robot description, xacro)
@@ -36,5 +36,5 @@
             <tf_topic>/tf</tf_topic>
             <dimensions>2</dimensions>
-            <odom_publish_frequency>10</odom_publish_frequency>
+            <odom_publish_frequency>100</odom_publish_frequency>
         </plugin>
     </gazebo>

File: models/prometheus/urdf/prometheus.xacro (robot description, xacro)
@@ -18,5 +18,5 @@
     <xacro:property name="traction_wheel_radius" value="0.05"/>
     <xacro:property name="traction_wheel_width" value="0.03"/>
-    <xacro:property name="traction_track_width" value="0.6"/>
+    <xacro:property name="traction_track_width" value="0.4"/>
     <xacro:property name="two_d_lidar_update_rate" value="30"/>
     <xacro:property name="two_d_lidar_sample_size" value="361"/>
